File: ExpressLRS-Nano-Receiver.kicad_sch (KiCad schematic)
At the start: 25 parts

Commit message: Finished PCB
Parts:
- added C14, C15: 10nF, Capacitor_SMD:C_0402_1005Metric, symbol Device:C
- added C16: 470nF, Capacitor_SMD:C_0402_1005Metric, symbol Device:C
- added C17, C18: 0.1uF, Capacitor_SMD:C_0402_1005Metric, symbol Device:C
- added C19: ~, Capacitor_SMD:C_0402_1005Metric, symbol Device:C
- added D1: LED, LED_SMD:LED_0402_1005Metric, symbol Device:LED
- added E1: NN02-201, Library:XCVR_NN02-201, symbol NN02-101:NN02-101
- added FL1: 2450FM07D0034T, Library:FIL_2450FM07D0034T, symbol 2450FM07D0034T:2450FM07D0034T
- added J1: CONN, Connector_PinHeader_2.54mm:PinHeader_1x04_P2.54mm_Vertical, symbol Connector:Conn_01x04_Pin
- added R8: 300R, Resistor_SMD:R_0402_1005Metric, symbol Device:R_Small
- added R9: 1K, Resistor_SMD:R_0402_1005Metric, symbol Device:R_Small
- added Y2: 52MHz, Crystal:Crystal_SMD_2016-4Pin_2.0x1.6mm, symbol Device:Crystal_GND24
- AE1: renamed from AE?; footprint (none) -> Library:esp-antenna
- U3: renamed from U?; Manufacturer (none) -> Semtech; Package-Case (none) -> QFN-24; Suplier (none) -> Mouser; Suplier Part Number (none) -> 947-SX1280IMLTRT; URL (none) -> https://www.mouser.com.tr/ProductDetail/Semtech/SX1280IMLTR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
- gave numbers to parts that had none: 23
Connections:
- net +3V3: now also U3.11 (VBAT_IO), U3.15 (VBAT), C17.1, C18.1, R8.2
- net +5V: now also J1.2 (Pin_2)
- net EPAD: now also C12.2, C9.2, U3.13 (GND), U3.20 (GND), U3.21 (GND), U3.23 (GND), U3.24 (GND), U3.25 (GND), U3.5 (GND), C14.1, C15.1, C16.2, C17.2, C18.2, C19.2, FL1.2, FL1.4, J1.1 (Pin_1), R9.1, Y2.2, Y2.4
- net MISO: now reaches U2.10 (MTDI)
- net MISO: now also U3.16 (MISO_TX)
- net MOSI: now reaches U2.12 (MTCK)
- net MOSI: now also U3.17 (MOSI_RX)
- net NSS: now reaches R1.2, U2.13 (MTDO)
- net NSS: now also U3.19 (NSS_CTS)
- net nRST: now reaches R4.2, U2.14 (GPIO2)
- net nRST: now also U3.3 (NRESET)
- net BTN: now reaches R2.1, U2.15 (GPIO0)
- net BTN: now also C19.1
- net DIO1: now reaches U2.16 (GPIO4)
- net DIO1: now also U3.8 (DIO1)
- net BUSY: now reaches U2.24 (GPIO5)
- net BUSY: now also U3.7 (BUSY)
- net RX: now reaches U2.25 (U0RXD)
- net RX: now also J1.4 (Pin_4)
- net TX: now reaches U2.26 (U0TXD)
- net TX: now also J1.3 (Pin_3), R8.1
- net LED: now reaches U2.8 (XPD_DCDC)
- net LED: now also D1.2 (A)
- net SCK: now reaches U2.9 (MTMS)
- net SCK: now also U3.18 (SCK_RTSN)
- net at U3.1 (VR_PA): now also C14.2
- net at U3.12 (DCC_FB): now also C16.1
- net at U3.2 (VDD_INN): now also C15.2
- net at U3.22 (RFIO): now also FL1.1
- net at U3.4 (XTA): now also Y2.3
- net at U3.6 (XTB): now also Y2.1
- new net: E1.1, FL1.3
- new net: D1.1 (K), R9.2
- no-connect marks 14 -> 11
Other:
- company: (none) -> Kolamuc Design
- title: (none) -> ExpressLRS Nano Receiver
- moved on the sheet: U3

Commit message: update
Parts:
- removed C16: 470nF, Capacitor_SMD:C_0402_1005Metric, symbol Device:C
- removed C19: ~, Capacitor_SMD:C_0402_1005Metric, symbol Device:C
- removed C7: 4.7uF, Capacitor_SMD:C_0402_1005Metric, symbol Device:C
- removed J1: CONN, Connector_PinHeader_2.54mm:PinHeader_1x04_P2.54mm_Vertical, symbol Connector:Conn_01x04_Pin
- removed R7: 100K, Resistor_SMD:R_0402_1005Metric, symbol Device:R_Small
- removed U1: TPS73533DRVR, Package_SON:WSON-6-1EP_2x2mm_P0.65mm_EP1x1.6mm, symbol Alperen:TPS73533DRVR
- added C20, C21: 2.2uF, Capacitor_SMD:C_0402_1005Metric, symbol Device:C
- added J1: Conn_01x05_Pin, Connector_PinHeader_2.00mm:PinHeader_1x05_P2.00mm_Vertical, symbol Connector:Conn_01x05_Pin
- added L1: 15uH, Inductor_SMD:L_0805_2012Metric, symbol Device:L_Small
- added U4: AP2210N-3.3TRG1, Package_TO_SOT_SMD:SOT-23-3, symbol AP2210N:AP2210N-3.3TRG1
- C1: value 2.2uF -> 470nF; Suplier Part Number CL05A225MQ5NNNC -> CL05A474KQ5NNNC; URL https://ozdisan.com/pasif-komponentler/kapasitorler/smt-smd-ve-mlcc-kapasitorler/CL05A225MQ5NNNC/521876 -> https://ozdisan.com/pasif-komponentler/kapasitorler/smt-smd-ve-mlcc-kapasitorler/CL05A474KQ5NNNC/518804
- C2: value 10nF -> 18pF; Suplier Part Number CL05B103KB5NNNC -> CL05C180JB5NNNC; URL https://ozdisan.com/pasif-komponentler/kapasitorler/smt-smd-ve-mlcc-kapasitorler/CL05B103KB5NNNC/30282 -> https://ozdisan.com/pasif-komponentler/kapasitorler/smt-smd-ve-mlcc-kapasitorler/CL05C180JB5NNNC/429001
- C5: value 0.1uF -> 18pF; Suplier Part Number CL05B104KO5NNNC -> CL05C180JB5NNNC; URL https://ozdisan.com/pasif-komponentler/kapasitorler/smt-smd-ve-mlcc-kapasitorler/CL05B104KO5NNNC/336698 -> https://ozdisan.com/pasif-komponentler/kapasitorler/smt-smd-ve-mlcc-kapasitorler/CL05C180JB5NNNC/429001
- Y1: footprint Crystal:Crystal_SMD_EuroQuartz_X22-4Pin_2.5x2.0mm -> Crystal:Crystal_SMD_2016-4Pin_2.0x1.6mm; Manufacturer RALTRON -> (none); Package-Case SMD -> 2016; Suplier Ozdisan -> (none); Suplier Part Number R2520-26.000-18-F-1010-E -> (none); URL https://ozdisan.com/pasif-komponentler/kristaller-osilatorl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 -> (none)
Connections:
- net +3V3: now also C21.1, U4.2 (VOUT); no longer C1.2
- net +5V: now also C20.2, J1.3 (Pin_3), U4.3 (VIN); no longer C5.1
- net BTN: now also J1.1 (Pin_1)
- net RX: now also J1.4 (Pin_4)
- net TX: now also J1.5 (Pin_5)
- net at C10.1: now also U2.28 (XTAL_IN), Y1.1; no longer Y1.2
- net at U2.27 (XTAL_OUT), Y1.3: now also C13.1
- net V_DCC: now reaches U3.12 (DCC_FB)
- net V_DCC: now also C1.1, C15.2, U3.2 (VDD_INN), L1.1
- net GND: now reaches C2.1
- net GND: now also AE1.2, C1.2, C10.2, C12.2, C13.2, C14.1, C15.1, C17.2, C18.2, C3.1, C4.2, C5.1, C6.2, C8.2, C9.2, FL1.2, FL1.4, R1.1, R5.2, R9.1, U2.33 (GND), U3.13 (GND), U3.20 (GND), U3.21 (GND), U3.23 (GND), U3.24 (GND), U3.25 (GND), U3.5 (GND), Y1.2, Y1.4, Y2.2, Y2.4, C20.1, C21.2, J1.2 (Pin_2), U4.1 (GND)
- net at U3.6 (XTB), Y2.1: now also C5.2
- net at U3.4 (XTA), Y2.3: now also C2.2
- net V_DCC2: now reaches U3.14 (DCC_SW)
- net V_DCC2: now also L1.2
- removed net EPAD: AE1.2, C1.1, C10.2, C12.2, C13.2, C14.1, C15.1, C17.2, C18.2, C2.2, C3.1, C4.2, C5.2, C6.2, C8.2, C9.2, FL1.2, FL1.4, R1.1, R5.2, R9.1, U2.33 (GND), U3.13 (GND), U3.20 (GND), U3.21 (GND), U3.23 (GND), U3.24 (GND), U3.25 (GND), U3.5 (GND), Y2.2, Y2.4
- no-connect marks 11 -> 10
Other:
- moved on the sheet: C10, C13, C17, C8
